File: ControlBoard.sch (EAGLE design)
At the start: 4 parts

Commit message: Added FT232 and button connectors.
Parts:
- removed SPI: CONNECTOR_6PIN2X3_ISP, connectors:CONNECTOR_6PIN2X3_ISP
- added BTNCON1, BTNCON2, BTNCON3, BTNCON4, BTNCON5, BTNCON6: CONNECTOR_2PIN1X2_WIRE, connectors:CONNECTOR_2PIN1X2_WIRE
- added C1, C2, C3: 100nF, RC_and_L:C-EUC0805
- added C4: 10nF, RC_and_L:C-EUC0805
- added FERRITE0: (no value), RC_and_L:R-EU_R0805
- added IC1: FT232RL, jogwheelParts:FT232RL
- added ISP: CONNECTOR_6PIN2X3_ISP, connectors:CONNECTOR_6PIN2X3_ISP
- added JOYSTICK2: JOYSTIC-XYRKJXK122000D, jogwheelParts:JOYSTIC-XYRKJXK122000D
- renumbered U$1 to JOYSTICK1
Connections:
- removed net N$1: JOYSTICK1.X3, JOYSTICK1.Y3
- removed net N$4: DEBUG.P$3, SPI.P$6
- removed net N$5: U$2.VCC, U$2.VCC@1, U$2.VCC@2
- new net +5V: C2.1, C4.1, FERRITE0.2, IC1.VCC, IC1.VCCIO, ISP.P$1, JOYSTICK1.X1, JOYSTICK1.Y1, JOYSTICK2.X1, JOYSTICK2.Y1, U$2.VCC, U$2.VCC@1, U$2.VCC@2
- new net GND: BTNCON1.P$1, BTNCON2.P$1, BTNCON3.P$1, BTNCON4.P$1, BTNCON5.P$1, BTNCON6.P$1, C1.2, C2.2, C3.1, C3.2, C4.2, DEBUG.P$3, IC1.AGND, IC1.GND@0, IC1.GND@1, IC1.GND@2, IC1.TEST, ISP.P$6, JOYSTICK1.X3, JOYSTICK1.Y3, JOYSTICK2.X3, JOYSTICK2.Y3, U$2.GND, U$2.GND@1, U$2.GND@2, U$2.GND@3
- new net N$10: C1.1, IC1.3V3OUT
- new net N$6: IC1.USBDP
- new net N$7: IC1.USBDM
- new net N$8: FERRITE0.1
- net !RESET: now also ISP.P$4; no longer SPI.P$4
- net N$2: now also IC1.CBUS0; no longer JOYSTICK1.X1, JOYSTICK1.Y1
- net N$3: now also IC1.CBUS1; no longer SPI.P$1
- net PORTA2: now also JOYSTICK2.Y2
- net PORTA3: now also JOYSTICK2.X2
- net PORTB5: now also ISP.P$3; no longer SPI.P$3
- net PORTB6: now also ISP.P$2; no longer SPI.P$2
- net PORTB7: now also ISP.P$5; no longer SPI.P$5
- net PORTC0: now also BTNCON1.P$2
- net PORTC1: now also BTNCON2.P$2
- net PORTC2: now also BTNCON3.P$2
- net PORTC3: now also BTNCON4.P$2
- net PORTC4: now also BTNCON5.P$2
- net PORTC5: now also BTNCON6.P$2
- net PORTD2: now also IC1.TXD
- net PORTD3: now also IC1.RXD
Other:
- moved on the sheet: DEBUG

Commit message: Added reference for ACD and USB connector.
Parts:
- added C5, C6: 22uF, RC_and_L:C-EUC1206
- added C7: 100nF, RC_and_L:C-EUC0805
- added CON1: USB-BWUERTH-ELECTRONIC-USB-B, jogwheelParts:USB-BWUERTH-ELECTRONIC-USB-B
- added L1: (no value), RC_and_L:L-USL0805
- added R1, R2: 1k, RC_and_L:R-EU_R0805
Connections:
- new net N$1: C7.2, U$2.AREF, U$2.AVCC
- new net N$5: C7.1, L1.2
- net +5V: now also C3.1, C6.1, L1.1
- net GND: now also C6.2, CON1.GND, CON1.SHIELD@1, CON1.SHIELD@2; no longer C3.1
- net N$2: now also R1.1
- net N$3: now also R2.1
- net N$6: now also CON1.D+
- net N$7: now also CON1.D-
- net N$8: now also CON1.VCC@1
Other:
- moved on the sheet: C3

Commit message: Added leds to RXD/TXD->USB
Parts:
- added U$1, U$3: LED, jogwheelParts:LED
- BTNCON1, BTNCON2, BTNCON3, BTNCON4, BTNCON5, BTNCON6, C5, C6, CON1, DEBUG, FERRITE0, IC1, ISP, JOYSTICK1, JOYSTICK2, L1, R1, R2, U$2: OC_NEWARK (none) -> unknown
- C1, C2, C3, C7: MF (none) -> FARNELL; MPN (none) -> KP-2012SEC; OC_NEWARK (none) -> 38K3382
- C4: MPN (none) -> 04023D103KAT2A; OC_NEWARK (none) -> 50R8273
Connections:
- new net N$4: R1.2, U$1.K
- new net N$9: R2.2, U$3.K
- net +5V: now also U$1.A, U$3.A

Commit message: Layout sketch done.
Parts:
- renumbered U$1 to RX, U$3 to TX
Changed lines of the file:
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@@
 <attribute name="OC_NEWARK" value="unknown"/>
 </part>
-<part name="U$1" library="jogwheelParts" deviceset="LED" device=""/>
-<part name="U$3" library="jogwheelParts" deviceset="LED" device=""/>
+<part name="RX" library="jogwheelParts" deviceset="LED" device=""/>
+<part name="TX" library="jogwheelParts" deviceset="LED" device=""/>
 <part name="P+7" library="schematic_supply" deviceset="+5V" device=""/>
 </parts>
@@
 <attribute name="MPN" x="-48.26" y="25.4" size="1.778" layer="96" display="off"/>
 </instance>
-<instance part="U$1" gate="G$1" x="-254" y="5.08" rot="R180"/>
-<instance part="U$3" gate="G$1" x="-243.84" y="5.08" rot="R180"/>
+<instance part="RX" gate="G$1" x="-254" y="5.08" rot="R180"/>
+<instance part="TX" gate="G$1" x="-243.84" y="5.08" rot="R180"/>
 <instance part="P+7" gate="1" x="-254" y="25.4"/>
 </instances>
@@
 </segment>
 <segment>
-<pinref part="U$3" gate="G$1" pin="A"/>
+<pinref part="TX" gate="G$1" pin="A"/>
 <wire x1="-243.84" y1="10.16" x2="-243.84" y2="15.24" width="0.1524" layer="91"/>
 <wire x1="-243.84" y1="15.24" x2="-254" y2="15.24" width="0.1524" layer="91"/>
-<pinref part="U$1" gate="G$1" pin="A"/>
+<pinref part="RX" gate="G$1" pin="A"/>
 <wire x1="-254" y1="15.24" x2="-254" y2="10.16" width="0.1524" layer="91"/>
 <wire x1="-254" y1="15.24" x2="-254" y2="20.32" width="0.1524" layer="91"/>
@@
 <net name="N$4" class="0">
 <segment>
-<pinref part="U$1" gate="G$1" pin="K"/>
+<pinref part="RX" gate="G$1" pin="K"/>
 <pinref part="R1" gate="G$1" pin="2"/>
 <wire x1="-254" y1="0" x2="-254" y2="-5.08" width="0.1524" layer="91"/>
@@
 <net name="N$9" class="0">
 <segment>
-<pinref part="U$3" gate="G$1" pin="K"/>
+<pinref part="TX" gate="G$1" pin="K"/>
 <pinref part="R2" gate="G$1" pin="2"/>
 <wire x1="-243.84" y1="0" x2="-243.84" y2="-5.08" width="0.1524" layer="91"/>
